File: kicad/controller/controller.kicad_sch (KiCad schematic)
At the start: 10 parts, among them J1 Conn_01x07_Male, U1 BluePill_STM32F103C

Commit message: work on kicad
Parts:
- added C3, C4, C5, C6, C7, C8, C9: C, Capacitor_SMD:C_0805_2012Metric, symbol Device:C
- added J2, J3, J4: Conn_01x07_Male, Connector_PinHeader_2.54mm:PinHeader_1x07_P2.54mm_Vertical, symbol Connector:Conn_01x07_Male
- added J_Boost1: Conn_01x03_Male, Connector_PinHeader_2.54mm:PinHeader_1x03_P2.54mm_Vertical, symbol Connector:Conn_01x03_Male
- added J_Button1: Conn_01x05_Male, Connector_PinHeader_2.54mm:PinHeader_1x05_P2.54mm_Vertical, symbol Connector:Conn_01x05_Male
- added J_Display1, J_SD1: Conn_01x04_Male, Connector_PinHeader_2.54mm:PinHeader_1x04_P2.54mm_Vertical, symbol Connector:Conn_01x04_Male
- added R10, R11, R12, R13, R14, R15, R16, R17, R18, R19, R20, R21, R22, R23, R24, R25, R26, R27, R28, R29, R30, R31, R32, R33, R7, R8, R9: 10k, Resistor_SMD:R_1206_3216Metric, symbol Device:R
- added U2: LM324, Package_SO:SOIC-14_3.9x8.7mm_P1.27mm, symbol Amplifier_Operational:LM324
Connections:
- net +12V: now also J2.1 (Pin_1), J3.1 (Pin_1), J4.1 (Pin_1), J_Boost1.3 (Pin_3)
- net A1: now also U1.5 (PA0); no longer U1.PA0
- net A2: now also U1.6 (PA1); no longer U1.PA1
- net GND: now also U1.19 (GND), U1.20 (GND), U1.39 (GND), C3.1, C4.2, C5.2, C6.2, C7.2, C8.2, C9.2, J2.3 (Pin_3), J3.3 (Pin_3), J4.3 (Pin_3), J_Boost1.2 (Pin_2), J_Button1.1 (Pin_1), J_Display1.1 (Pin_1), R14.2, R15.2, R16.2, R17.2, R18.2, R19.2, U2.11 (V-)
- net IN1: now also R26.2
- net IN2: now also R27.2
- net PWM1: now also U1.25 (PA8); no longer U1.PA8
- net PWM2: now also U1.26 (PA9_TX1); no longer U1.PA9 (PA9_TX1)
- net A6: now reaches U1.10 (PA5_SCK1)
- net A6: now also R11.1, R17.1
- net A7: now reaches U1.11 (PA6_MISO1)
- net A7: now also R12.1, R18.1
- net A8: now reaches U1.12 (PA7_MOSI1)
- net A8: now also R13.1, R19.1
- net REF_IN: now reaches U1.15 (PB10_SCL2)
- net REF_IN: now also R7.1
- net PWM4: now reaches U1.16 (PB11_SDA2)
- net PWM4: now also R21.2
- net +3.3V: now reaches U1.18 (VCC3V3)
- net +3.3V: now also U1.40 (VCC3V3), J_Button1.2 (Pin_2), U2.4 (V+)
- net at U1.21 (PB12): now also J_SD1.1 (Pin_1)
- net at U1.22 (PB13_SCK2): now also J_SD1.2 (Pin_2)
- net at U1.23 (PB14_MISO2): now also J_SD1.3 (Pin_3)
- net at U1.24 (PB15_MOSI2): now also J_SD1.4 (Pin_4)
- net PWM3: now reaches U1.27 (PA10_RX1)
- net PWM3: now also R20.2
- net SW: now reaches U1.3 (PC14)
- net SW: now also J_Button1.3 (Pin_3)
- net PWM5: now reaches U1.30 (PA15)
- net PWM5: now also R22.2
- net PWM6: now reaches U1.31 (PB3)
- net PWM6: now also R23.2
- net PWM7: now reaches U1.32 (PB4)
- net PWM7: now also R24.2
- net PWM8: now reaches U1.33 (PB5)
- net PWM8: now also R25.2
- net at U1.34 (PB6_SCL1): now also J_Display1.4 (Pin_4)
- net SDA: now reaches U1.35 (PB7_SDA1)
- net SDA: now also J_Display1.3 (Pin_3)
- net CLK: now reaches U1.36 (PB8)
- net CLK: now also J_Button1.5 (Pin_5)
- net DT: now reaches U1.37 (PB9)
- net DT: now also J_Button1.4 (Pin_4)
- net +5V: now reaches U1.38 (5V_USB)
- net +5V: now also J_Boost1.1 (Pin_1), J_Display1.2 (Pin_2)
- net A3: now reaches U1.7 (PA2_TX2)
- net A3: now also R14.1, R8.1
- net A4: now reaches U1.8 (PA3_RX2)
- net A4: now also R15.1, R9.1
- net A5: now reaches U1.9 (PA4)
- net A5: now also R10.1, R16.1
- net ref renamed ref1
- net ref1: now also R26.1, R27.1, U2.1, U2.2 (-)
- new net: C3.2, R7.2, U2.10 (+), U2.12 (+), U2.3 (+), U2.5 (+)
- new net IN3: C4.1, J2.4 (Pin_4), R20.1, R28.2
- new net IN4: C5.1, J2.6 (Pin_6), R21.1, R29.2
- new net IN5: C6.1, J3.4 (Pin_4), R22.1, R30.2
- new net IN6: C7.1, J3.6 (Pin_6), R23.1, R31.2
- new net IN7: C8.1, J4.4 (Pin_4), R24.1, R32.2
- new net IN8: C9.1, J4.6 (Pin_6), R25.1, R33.2
- new net U3: J2.5 (Pin_5), R8.2
- new net U4: J2.7 (Pin_7), R9.2
- new net U5: J3.5 (Pin_5), R10.2
- new net U6: J3.7 (Pin_7), R11.2
- new net U7: J4.5 (Pin_5), R12.2
- new net U8: J4.7 (Pin_7), R13.2
- new net ref2: J2.2 (Pin_2), R28.1, R29.1, U2.6 (-), U2.7
- new net ref3: J3.2 (Pin_2), R30.1, R31.1, U2.13 (-), U2.14
- new net ref4: J4.2 (Pin_2), R32.1, R33.1, U2.8, U2.9 (-)
Other:
- moved on the sheet: C2, J1, R6

Commit message: rework PINS, get SD Card working
Parts:
- added C10, C11, C12, C13, C14, C15, C16, C17, C18, C19, C20, C21: C, Capacitor_SMD:C_0805_2012Metric, symbol Device:C
- J_SD1: value Conn_01x04_Male -> Conn_01x06_Male; footprint Connector_PinHeader_2.54mm:PinHeader_1x04_P2.54mm_Vertical -> controller:SD_Card_reader; symbol Connector:Conn_01x04_Male -> Connector:Conn_01x06_Male
Connections:
- net +3.3V: now also J_SD1.1 (Pin_1), C19.2, C20.2, C21.2
- net +5V: now also C18.2
- net A1: now also C10.1
- net A2: now also C11.1
- net A3: now also C12.1
- net A4: now also C13.1
- net A5: now also C14.1
- net A6: now also C15.1
- net A7: now also C16.1
- net A8: now also C17.1
- net GND: now also J_SD1.6 (Pin_6), C10.2, C11.2, C12.2, C13.2, C14.2, C15.2, C16.2, C17.2, C18.1, C19.1, C20.1, C21.1
- net PWM3: now also U1.16 (PB11_SDA2); no longer U1.27 (PA10_RX1)
- net PWM4: now also U1.14 (PB1); no longer U1.16 (PB11_SDA2)
- net PWM5: now also U1.27 (PA10_RX1); no longer U1.30 (PA15)
- net PWM6: now also U1.30 (PA15); no longer U1.31 (PB3)
- net PWM7: now also U1.31 (PB3); no longer U1.32 (PB4)
- net PWM8: now also U1.32 (PB4); no longer U1.33 (PB5)
- net SW: now also U1.33 (PB5); no longer U1.3 (PC14)
- net ref1: no longer R26.1, R27.1
- net ref2: now also R26.1, R27.1
- net at U1.21 (PB12): now also J_SD1.2 (Pin_2); no longer J_SD1.1 (Pin_1)
- net at U1.22 (PB13_SCK2): now also J_SD1.4 (Pin_4); no longer J_SD1.2 (Pin_2)
- net at J_SD1.3 (Pin_3): now also U1.24 (PB15_MOSI2); no longer U1.23 (PB14_MISO2)
- new net: J_SD1.5 (Pin_5), U1.23 (PB14_MISO2)
Other:
- moved on the sheet: R10, R11, R12, R13, R14, R15, R16, R17, R18, R19, R2, R4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

Commit message: work on kicad
Parts:
- added J_PWR1: Conn_01x02_Male, Connector_PinHeader_2.54mm:PinHeader_1x02_P2.54mm_Vertical, symbol Connector:Conn_01x02_Male
Connections:
- net +5V: now also J_PWR1.1 (Pin_1)
- net GND: now also J_PWR1.2 (Pin_2)
Changed lines of the file:
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@@
+    (stroke (width 0) (type default) (color 0 0 0 0))
+  )
+  (wire (pts (xy 119.38 38.1) (xy 124.46 38.1))
     (stroke (width 0) (type default) (color 0 0 0 0))
   )
@@
   )
   (wire (pts (xy 214.63 29.21) (xy 215.9 29.21))
+    (stroke (width 0) (type default) (color 0 0 0 0))
+  )
+  (wire (pts (xy 119.38 35.56) (xy 124.46 35.56))
     (stroke (width 0) (type default) (color 0 0 0 0))
   )
@@
     (pin "2")
   )
+  (symbol (lib_id "power:+5V") (at 124.46 35.56 270) (unit 1)
+    (in_bom yes) (on_board yes) (fields_autoplaced)
+    (property "Reference" "#PWR0147" (id 0) (at 120.65 35.56 0)
+      (effects (font (size 1.27 1.27)) hide)
+    )
+    (property "Value" "+5V" (id 1) (at 128.27 35.5599 90)
+      (effects (font (size 1.27 1.27)) (justify left))
+    )
+    (property "Footprint" "" (id 2) (at 124.46 35.56 0)
+      (effects (font (size 1.27 1.27)) hide)
+    )
+    (property "Datasheet" "" (id 3) (at 124.46 35.56 0)
+      (effects (font (size 1.27 1.27)) hide)
+    )
+    (pin "1")
+  )
   (symbol (lib_id "Device:R") (at 210.82 39.37 90) (unit 1)
     (in_bom yes) (on_board yes)
@@
     (pin "1")
   )
+  (symbol (lib_id "power:GND") (at 124.46 38.1 90) (unit 1)
+    (in_bom yes) (on_board yes) (fields_autoplaced)
+    (property "Reference" "#PWR0146" (id 0) (at 130.81 38.1 0)
+      (effects (font (size 1.27 1.27)) hide)
+    )
+    (property "Value" "GND" (id 1) (at 128.27 38.0999 90)
+      (effects (font (size 1.27 1.27)) (justify right))
+    )
+    (property "Footprint" "" (id 2) (at 124.46 38.1 0)
+      (effects (font (size 1.27 1.27)) hide)
+    )
+    (property "Datasheet" "" (id 3) (at 124.46 38.1 0)
+      (effects (font (size 1.27 1.27)) hide)
+    )
+    (pin "1")
+  )
   (symbol (lib_id "Device:C") (at 148.59 44.45 180) (unit 1)
     (in_bom yes) (on_board yes) (fields_autoplaced)
@@
     (pin "2")
     (pin "3")
+  )
+  (symbol (lib_id "Connector:Conn_01x02_Male") (at 114.3 35.56 0) (unit 1)
+    (in_bom yes) (on_board yes)
+    (property "Reference" "J_PWR1" (id 0) (at 114.3 34.29 0))
+    (property "Value" "Conn_01x02_Male" (id 1) (at 114.3 41.91 0))
+    (property "Footprint" "Connector_PinHeader_2.54mm:PinHeader_1x02_P2.54mm_Vertical" (id 2) (at 114.3 35.56 0)
+      (effects (font (size 1.27 1.27)) hide)
+    )
+    (property "Datasheet" "~" (id 3) (at 114.3 35.56 0)
+      (effects (font (size 1.27 1.27)) hide)
+    )
+    (pin "1")
+    (pin "2")
   )
   (symbol (lib_id "controller:BluePill_STM32F103C") (at 124.46 101.6 0) (unit 1)
@@
       (reference "#PWR0145") (unit 1) (value "GND") (footprint "")
     )
+    (path "/e041ddf6-511e-46b5-85e7-48f94616420f"
+      (reference "#PWR0146") (unit 1) (value "GND") (footprint "")
+    )
+    (path "/8ec97c68-04eb-48c6-9690-1f14051e386c"
+      (reference "#PWR0147") (unit 1) (value "+5V") (footprint "")
+    )
     (path "/33fbdfb4-0ded-49b6-9d3b-34389180e4ea"
       (reference "C1") (unit 1) (value "C") (footprint "Capacitor_SMD:C_0805_2012Metric")
@@
       (reference "J_Display1") (unit 1) (value "Conn_01x04_Male") (footprint "Connector_PinHeader_2.54mm:PinHeader_1x04_P2.54mm_Vertical")
     )
+    (path "/f91cfb3c-6975-4a90-81a5-9157eb0c254c"
+      (reference "J_PWR1") (unit 1) (value "Conn_01x02_Male") (footprint "Connector_PinHeader_2.54mm:PinHeader_1x02_P2.54mm_Vertical")
+    )
     (path "/808e8c67-5046-43e2-af3a-ef81f2b327bd"
