File: kicad/channel2/channel2.kicad_sch (KiCad schematic)
At the start: 43 parts, among them J1 Conn_01x07_Male, J5V1 Conn_01x01_Male, Q1 BC846B, Q2 IRF3205, Q3 IRF3205, Q4 BC846B, Q5 IRF3205, Q6 IRF3205, U1 LM324

Commit message: work on pulse charge/discharge, combined board
Parts:
- added JTest1, JTest2: Conn_01x01_Male, Connector_PinHeader_2.54mm:PinHeader_1x01_P2.54mm_Vertical, symbol Connector:Conn_01x01_Male
Connections:
- net GND1: now reaches JGND1.1 (Pin_1), Q6.3 (S)
- net GND2: now reaches JGND2.1 (Pin_1), Q3.3 (S)
- net at Q1.1 (B), R6.1: now also JTest2.1 (Pin_1)
- net at Q4.1 (B), R14.1: now also JTest1.1 (Pin_1)
Changed lines of the file:
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@@
   (junction (at 152.4 132.08) (diameter 0) (color 0 0 0 0)
   )
+  (junction (at 146.05 59.69) (diameter 0) (color 0 0 0 0)
+  )
   (junction (at 167.64 121.92) (diameter 0) (color 0 0 0 0)
   )
@@
   (junction (at 128.27 33.02) (diameter 0) (color 0 0 0 0)
   )
+  (junction (at 138.43 134.62) (diameter 0) (color 0 0 0 0)
+  )
   (junction (at 91.44 118.11) (diameter 0) (color 0 0 0 0)
   )
@@
     (stroke (width 0) (type default) (color 0 0 0 0))
   )
-  (wire (pts (xy 146.05 55.88) (xy 146.05 60.96))
+  (wire (pts (xy 146.05 55.88) (xy 146.05 59.69))
     (stroke (width 0) (type default) (color 0 0 0 0))
   )
@@
     (stroke (width 0) (type default) (color 0 0 0 0))
   )
-  (wire (pts (xy 138.43 132.08) (xy 138.43 137.16))
+  (wire (pts (xy 138.43 132.08) (xy 138.43 134.62))
     (stroke (width 0) (type default) (color 0 0 0 0))
   )
@@
     (stroke (width 0) (type default) (color 0 0 0 0))
   )
+  (wire (pts (xy 153.67 33.02) (xy 167.64 33.02))
+    (stroke (width 0) (type default) (color 0 0 0 0))
+  )
   (wire (pts (xy 110.49 118.11) (xy 110.49 149.86))
     (stroke (width 0) (type default) (color 0 0 0 0))
@@
     (stroke (width 0) (type default) (color 0 0 0 0))
   )
+  (wire (pts (xy 138.43 134.62) (xy 138.43 137.16))
+    (stroke (width 0) (type default) (color 0 0 0 0))
+  )
   (wire (pts (xy 142.24 36.83) (xy 142.24 33.02))
     (stroke (width 0) (type default) (color 0 0 0 0))
@@
     (stroke (width 0) (type default) (color 0 0 0 0))
   )
-  (wire (pts (xy 26.67 92.71) (xy 31.75 92.71))
+  (wire (pts (xy 26.67 92.71) (xy 33.02 92.71))
     (stroke (width 0) (type default) (color 0 0 0 0))
   )
@@
     (stroke (width 0) (type default) (color 0 0 0 0))
   )
+  (wire (pts (xy 146.05 59.69) (xy 146.05 60.96))
+    (stroke (width 0) (type default) (color 0 0 0 0))
+  )
+  (wire (pts (xy 146.05 132.08) (xy 152.4 132.08))
+    (stroke (width 0) (type default) (color 0 0 0 0))
+  )
+  (wire (pts (xy 201.93 45.72) (xy 201.93 73.66))
+    (stroke (width 0) (type default) (color 0 0 0 0))
+  )
+  (wire (pts (xy 232.41 102.87) (xy 232.41 105.41))
+    (stroke (width 0) (type default) (color 0 0 0 0))
+  )
+  (wire (pts (xy 43.18 71.12) (xy 62.23 71.12))
+    (stroke (width 0) (type default) (color 0 0 0 0))
+  )
   (wire (pts (xy 151.13 105.41) (xy 158.75 105.41))
-    (stroke (width 0) (type default) (color 0 0 0 0))
-  )
-  (wire (pts (xy 146.05 132.08) (xy 152.4 132.08))
-    (stroke (width 0) (type default) (color 0 0 0 0))
-  )
-  (wire (pts (xy 201.93 45.72) (xy 201.93 73.66))
-    (stroke (width 0) (type default) (color 0 0 0 0))
-  )
-  (wire (pts (xy 232.41 102.87) (xy 232.41 105.41))
-    (stroke (width 0) (type default) (color 0 0 0 0))
-  )
-  (wire (pts (xy 31.75 88.9) (xy 31.75 92.71))
-    (stroke (width 0) (type default) (color 0 0 0 0))
-  )
-  (wire (pts (xy 153.67 33.02) (xy 167.64 33.02))
-    (stroke (width 0) (type default) (color 0 0 0 0))
-  )
-  (wire (pts (xy 43.18 71.12) (xy 62.23 71.12))
     (stroke (width 0) (type default) (color 0 0 0 0))
   )
@@
     )
   )
-  (global_label "ref" (shape input) (at 38.1 95.25 90) (fields_autoplaced)
+  (global_label "ref" (shape input) (at 45.72 95.25 90) (fields_autoplaced)
     (effects (font (size 1.27 1.27)) (justify left))
-    (property "Intersheet References" "${INTERSHEET_REFS}" (id 0) (at 38.0206 90.2364 90)
+    (property "Intersheet References" "${INTERSHEET_REFS}" (id 0) (at 45.6406 90.2364 90)
       (effects (font (size 1.27 1.27)) (justify left) hide)
     )
@@
     )
   )
+  (global_label "GND1" (shape input) (at 175.26 71.12 0) (fields_autoplaced)
+    (effects (font (size 1.27 1.27)) (justify left))
+    (property "Intersheet References" "${INTERSHEET_REFS}" (id 0) (at 182.7531 71.0406 0)
+      (effects (font (size 1.27 1.27)) (justify left) hide)
+    )
+  )
   (global_label "U2" (shape input) (at 30.48 107.95 0) (fields_autoplaced)
     (effects (font (size 1.27 1.27)) (justify left))
@@
     (property "Intersheet References" "${INTERSHEET_REFS}" (id 0) (at 200.5806 126.8731 90)
       (effects (font (size 1.27 1.27)) (justify right) hide)
+    )
+  )
+  (global_label "GND2" (shape input) (at 167.64 147.32 0) (fields_autoplaced)
+    (effects (font (size 1.27 1.27)) (justify left))
+    (property "Intersheet References" "${INTERSHEET_REFS}" (id 0) (at 175.1331 147.2406 0)
+      (effects (font (size 1.27 1.27)) (justify left) hide)
     )
   )
@@
     (pin "1")
   )
-  (symbol (lib_id "power:+12V") (at 31.75 88.9 0) (unit 1)
-    (in_bom yes) (on_board yes) (fields_autoplaced)
-    (property "Reference" "#PWR0104" (id 0) (at 31.75 92.71 0)
-      (effects (font (size 1.27 1.27)) hide)
-    )
-    (property "Value" "+12V" (id 1) (at 31.75 83.82 0))
-    (property "Footprint" "" (id 2) (at 31.75 88.9 0)
-      (effects (font (size 1.27 1.27)) hide)
-    )
-    (property "Datasheet" "" (id 3) (at 31.75 88.9 0)
+  (symbol (lib_id "power:+12V") (at 33.02 92.71 270) (unit 1)
+    (in_bom yes) (on_board yes) (fields_autoplaced)
+    (property "Reference" "#PWR0104" (id 0) (at 29.21 92.71 0)
+      (effects (font (size 1.27 1.27)) hide)
+    )
+    (property "Value" "+12V" (id 1) (at 36.83 92.7099 90)
+      (effects (font (size 1.27 1.27)) (justify left))
+    )
+    (property "Footprint" "" (id 2) (at 33.02 92.71 0)
+      (effects (font (size 1.27 1.27)) hide)
+    )
+    (property "Datasheet" "" (id 3) (at 33.02 92.71 0)
       (effects (font (size 1.27 1.27)) hide)
     )
@@
     (pin "2")
   )
+  (symbol (lib_id "Connector:Conn_01x01_Male") (at 133.35 134.62 0) (unit 1)
+    (in_bom yes) (on_board yes)
+    (property "Reference" "JTest2" (id 0) (at 132.08 132.08 0))
+    (property "Value" "Conn_01x01_Male" (id 1) (at 133.35 137.16 0))
+    (property "Footprint" "Connector_PinHeader_2.54mm:PinHeader_1x01_P2.54mm_Vertical" (id 2) (at 133.35 134.62 0)
+      (effects (font (size 1.27 1.27)) hide)
+    )
+    (property "Datasheet" "~" (id 3) (at 133.35 134.62 0)
+      (effects (font (size 1.27 1.27)) hide)
+    )
+    (pin "1")
+  )
   (symbol (lib_id "Amplifier_Operational:LM324") (at 113.03 33.02 0) (unit 4)
     (in_bom yes) (on_board yes)
@@
     (pin "2")
   )
+  (symbol (lib_id "Connector:Conn_01x01_Male") (at 140.97 59.69 0) (unit 1)
+    (in_bom yes) (on_board yes)
+    (property "Reference" "JTest1" (id 0) (at 139.7 57.15 0))
+    (property "Value" "Conn_01x01_Male" (id 1) (at 140.97 62.23 0))
+    (property "Footprint" "Connector_PinHeader_2.54mm:PinHeader_1x01_P2.54mm_Vertical" (id 2) (at 140.97 59.69 0)
+      (effects (font (size 1.27 1.27)) hide)
+    )
+    (property "Datasheet" "~" (id 3) (at 140.97 59.69 0)
+      (effects (font (size 1.27 1.27)) hide)
+    )
+    (pin "1")
+  )
   (symbol (lib_id "Device:R") (at 118.11 149.86 90) (unit 1)
     (in_bom yes) (on_board yes)
@@
       (reference "JGND2") (unit 1) (value "Conn_01x01_Male") (footprint "Channel:PowerPad")
     )
+    (path "/d5522809-20fa-4999-9c02-30e06b1e4e14"
+      (reference "JTest1") (unit 1) (value "Conn_01x01_Male") (footprint "Connector_PinHeader_2.54mm:PinHeader_1x01_P2.54mm_Vertical")
+    )
+    (path "/ad5a32da-408f-48e0-8165-175f1e72feda"
+      (reference "JTest2") (unit 1) (value "Conn_01x01_Male") (footprint "Connector_PinHeader_2.54mm:PinHeader_1x01_P2.54mm_Vertical")
+    )
     (path "/4d794964-e9e6-43e9-ba42-f7ac638aaab0"

Commit message: fix resistor values around transistor
Parts:
- R14, R15, R6, R7: value 10k -> 22k
- R19, R20: value 2.2k -> 1k
Changed lines of the file:
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@@
       (effects (font (size 1.27 1.27)) (justify right))
     )
-    (property "Value" "2.2k" (id 1) (at 148.59 157.4799 0)
+    (property "Value" "1k" (id 1) (at 148.59 157.4799 0)
       (effects (font (size 1.27 1.27)) (justify right))
     )
@@
       (effects (font (size 1.27 1.27)) (justify right))
     )
-    (property "Value" "10k" (id 1) (at 154.94 123.1899 0)
+    (property "Value" "22k" (id 1) (at 154.94 123.1899 0)
       (effects (font (size 1.27 1.27)) (justify right))
     )
@@
       (effects (font (size 1.27 1.27)) (justify right))
     )
-    (property "Value" "10k" (id 1) (at 140.97 129.5399 0)
+    (property "Value" "22k" (id 1) (at 140.97 129.5399 0)
       (effects (font (size 1.27 1.27)) (justify right))
     )
@@
       (effects (font (size 1.27 1.27)) (justify right))
     )
-    (property "Value" "10k" (id 1) (at 148.59 53.3399 0)
+    (property "Value" "22k" (id 1) (at 148.59 53.3399 0)
       (effects (font (size 1.27 1.27)) (justify right))
     )
@@
       (effects (font (size 1.27 1.27)) (justify right))
     )
-    (property "Value" "2.2k" (id 1) (at 156.21 81.2799 0)
+    (property "Value" "1k" (id 1) (at 156.21 81.2799 0)
       (effects (font (size 1.27 1.27)) (justify right))
     )
@@
       (effects (font (size 1.27 1.27)) (justify right))
     )
-    (property "Value" "10k" (id 1) (at 162.56 46.9899 0)
+    (property "Value" "22k" (id 1) (at 162.56 46.9899 0)
       (effects (font (size 1.27 1.27)) (justify right))
     )
@@
     )
     (path "/9cdee3ab-c82d-4ff6-83b3-499badc4b793"
-      (reference "R6") (unit 1) (value "10k") (footprint "Resistor_SMD:R_1206_3216Metric")
+      (reference "R6") (unit 1) (value "22k") (footprint "Resistor_SMD:R_1206_3216Metric")
     )
     (path "/2fa500ec-a5b6-4fcc-8cfc-4d5ddf22cad7"
-      (reference "R7") (unit 1) (value "10k") (footprint "Resistor_SMD:R_1206_3216Metric")
+      (reference "R7") (unit 1) (value "22k") (footprint "Resistor_SMD:R_1206_3216Metric")
     )
     (path "/c800057a-d278-4182-854b-774312f90617"
@@
     )
     (path "/a0cacef5-f914-4b5f-aee2-b44c4a3e1231"
-      (reference "R14") (unit 1) (value "10k") (footprint "Resistor_SMD:R_1206_3216Metric")
+      (reference "R14") (unit 1) (value "22k") (footprint "Resistor_SMD:R_1206_3216Metric")
     )
     (path "/fcff7721-c065-4dc8-8503-125b039071bc"
-      (reference "R15") (unit 1) (value "10k") (footprint "Resistor_SMD:R_1206_3216Metric")
+      (reference "R15") (unit 1) (value "22k") (footprint "Resistor_SMD:R_1206_3216Metric")
     )
     (path "/e0875e71-84a2-420c-8418-813f497263e2"
@@
     )
     (path "/2d1ea026-a64f-45f8-b9b5-9a0b3db75686"
-      (reference "R19") (unit 1) (value "2.2k") (footprint "Resistor_SMD:R_1206_3216Metric")
+      (reference "R19") (unit 1) (value "1k") (footprint "Resistor_SMD:R_1206_3216Metric")
     )
     (path "/d43658fa-a692-4d09-9522-aaf7fd9b0d94"
-      (reference "R20") (unit 1) (value "2.2k") (footprint "Resistor_SMD:R_1206_3216Metric")
+      (reference "R20") (unit 1) (value "1k") (footprint "Resistor_SMD:R_1206_3216Metric")
     )
     (path "/29179f6f-ac0f-419e-9644-3e7dc970e2a3"
